File: kicad/12c508/midi-panic.sch (KiCad schematic (older format))
At the start: 17 parts

Commit message: Update schematics to KiCad 5. Update wks files.
Parts:
- removed R?: 220R, Resistors_SMD:R_1206_HandSoldering, symbol R
- removed R?: 1k2, Resistors_SMD:R_1206_HandSoldering, symbol R
- removed R?: 10k, Resistors_SMD:R_1206_HandSoldering, symbol R
- added R?: 220R, symbol Device:R_Small
- added R?: 10k, symbol Device:R_Small
- added R?: 1k2, symbol Device:R_Small
- C?: symbol C_Small -> midi-panic-rescue:C_Small
- C?: symbol CP1_Small -> midi-panic-rescue:CP1_Small
- D? (x2): symbol D_Small_ALT -> midi-panic-rescue:D_Small_ALT
- P? (x2): symbol DIN_5 -> midi-panic-rescue:DIN_5
- R? (x2): symbol R -> midi-panic-rescue:R
- SW? (x2): symbol PUSH_BUTTON-RESCUE-tinyVT -> midi-panic-rescue:PUSH_BUTTON-RESCUE-tinyVT
- SW? (x2): symbol SW_DPST_x2 -> midi-panic-rescue:SW_DPST_x2
- U?: symbol PIC12C508-I/P -> midi-panic-rescue:PIC12C508-I_P
- U?: symbol 6N136 -> midi-panic-rescue:6N136
Connections:
- wire segments 49 -> 61
Other:
- moved on the sheet: D?, P?, SW?, SW?A
